File: hardware/kicad/flowcontrol/sol2_output.kicad_sch (KiCad schematic)
At the start: 7 parts, among them J2 SOL2_PORT, Q2 SOL2_NPN

Commit message: Schemiatic update
Parts:
- removed Q2: SOL2_NPN, symbol Simulation_SPICE:NPN
- added Q3: SOL2_NFET, Package_TO_SOT_SMD:SOT-23, symbol Transistor_FET:MMBFJ113
- added R5: 10kO, Resistor_THT:R_Axial_DIN0309_L9.0mm_D3.2mm_P15.24mm_Horizontal, symbol Device:R
- added R6: 1kO, Resistor_THT:R_Axial_DIN0309_L9.0mm_D3.2mm_P15.24mm_Horizontal, symbol Device:R
- D3, D4: footprint (none) -> LED_THT:LED_Oval_W5.2mm_H3.8mm
- J2: footprint (none) -> Connector_PinSocket_2.00mm:PinSocket_1x02_P2.00mm_Vertical
- R2, R2LED_G1, R2LED_R1: footprint (none) -> Resistor_THT:R_Axial_DIN0309_L9.0mm_D3.2mm_P15.24mm_Horizontal
Connections:
- net 12V_IN: now also Q3.2 (S)
- net GND: now also R5.2
- net at J2.1 (Pin_1): now also Q3.1 (D)
- net at D3.1 (K), R2.2: now also R5.1, R6.1
- new net: Q3.3 (G), R6.2
Other:
- moved on the sheet: J2
