File: hardware/kicad/flowcontrol/flowcontrol.kicad_pcb (KiCad board)
At the start: 2 copper layers, 29 parts, among them J2 SOL2_PORT, J3 SOL1_PORT, Q1 SOL1_NFET, Q3 SOL2_NFET, SW10 SOL2_MASTER, SW3 SOL1_DURA, SW4 SOL1_DELAY, SW5 SOL2_DURA, SW6 SOL2_DELAY, SW9 SOL1_MASTER, U1 SOL1_DISP, U2 SOL2_DISP, U3 SOL1_AND_2 SPLIT, U4 XL1509-3.3

Commit message: semi-final updates for the report
Parts:
- removed R2LED_G1: 220, Resistor_THT:R_Axial_DIN0309_L9.0mm_D3.2mm_P15.24mm_Horizontal
- removed R2LED_R1: R, Resistor_THT:R_Axial_DIN0309_L9.0mm_D3.2mm_P15.24mm_Horizontal
- removed SW4: SOL1_DELAY, Rotary_Encoder:RotaryEncoder_Alps_EC11E_Vertical_H20mm
- removed SW9: SOL1_MASTER, Button_Switch_THT:SW_DIP_SPSTx01_Slide_6.7x4.1mm_W7.62mm_P2.54mm_LowProfile
- removed U2: SOL2_DISP, Display_7Segment:CA56-12SRWA
- removed U3: SOL1_AND_2 SPLIT, Package_DIP:DIP-28_W7.62mm
- added D1: SOL1_GRN, LED_THT:LED_Oval_W5.2mm_H3.8mm, F.Cu at (203.7, 54.2)
- added D2: SOL1_RED, LED_THT:LED_Oval_W5.2mm_H3.8mm, F.Cu at (187.2, 53.2)
- added J1: 4-digit I2C Display, Connector_PinHeader_2.54mm:PinHeader_1x04_P2.54mm_Vertical, F.Cu at (44.4, 64.4)
- added J4: SOL1_PORT, Connector_PinSocket_2.00mm:PinSocket_1x02_P2.00mm_Vertical, F.Cu at (276.0, 104.0)
- added Q2: SOL1_NFET, Package_TO_SOT_SMD:SOT-23, F.Cu at (216.6, 59.6)
- added R10: 100O, Resistor_THT:R_Axial_DIN0309_L9.0mm_D3.2mm_P15.24mm_Horizontal, F.Cu at (240.2, 72.5)
- added R11: 1kO, Resistor_THT:R_Axial_DIN0309_L9.0mm_D3.2mm_P15.24mm_Horizontal, F.Cu at (248.0, 77.7)
- added R12: 100, Resistor_THT:R_Axial_DIN0309_L9.0mm_D3.2mm_P15.24mm_Horizontal, F.Cu at (239.5, 78.4)
- added R1LED_G2: 220, Resistor_THT:R_Axial_DIN0309_L9.0mm_D3.2mm_P15.24mm_Horizontal, F.Cu at (206.8, 76.0)
- added R1LED_G3: 220, Resistor_THT:R_Axial_DIN0309_L9.0mm_D3.2mm_P15.24mm_Horizontal, F.Cu at (269.0, 75.7)
- added R1LED_R2: R, Resistor_THT:R_Axial_DIN0309_L9.0mm_D3.2mm_P15.24mm_Horizontal, F.Cu at (191.0, 75.6)
- added R1LED_R3: R, Resistor_THT:R_Axial_DIN0309_L9.0mm_D3.2mm_P15.24mm_Horizontal, F.Cu at (254.0, 77.2)
- added R7: 1kO, Resistor_THT:R_Axial_DIN0309_L9.0mm_D3.2mm_P15.24mm_Horizontal, F.Cu at (184.0, 75.5)
- added R8: 100, Resistor_THT:R_Axial_DIN0309_L9.0mm_D3.2mm_P15.24mm_Horizontal, F.Cu at (176.2, 75.6)
- added R9: 1kO, Resistor_THT:R_Axial_DIN0309_L9.0mm_D3.2mm_P15.24mm_Horizontal, F.Cu at (239.3, 100.5)
- added REF**: PinHeader_1x06_P2.54mm_Vertical, Connector_PinHeader_2.54mm:PinHeader_1x06_P2.54mm_Vertical, F.Cu at (188.0, 44.0)
- added REF**: PinHeader_1x06_P2.54mm_Vertical, Connector_PinHeader_2.54mm:PinHeader_1x06_P2.54mm_Vertical, F.Cu at (123.5, 44.0)
- added REF**: PinHeader_1x04_P2.54mm_Vertical, Connector_PinHeader_2.54mm:PinHeader_1x04_P2.54mm_Vertical, F.Cu at (41.3, 48.5)
- added REF**: PinHeader_1x04_P2.54mm_Vertical, Connector_PinHeader_2.54mm:PinHeader_1x04_P2.54mm_Vertical, F.Cu at (57.8, 48.5)
- added REF**: PinHeader_1x06_P2.54mm_Vertical, Connector_PinHeader_2.54mm:PinHeader_1x06_P2.54mm_Vertical, F.Cu at (257.0, 43.5)
- added REF**: PinHeader_1x04_P2.54mm_Vertical, Connector_PinHeader_2.54mm:PinHeader_1x04_P2.54mm_Vertical, F.Cu at (75.5, 48.5)
- added REF**: PinHeader_1x02_P2.54mm_Vertical, Connector_PinHeader_2.54mm:PinHeader_1x02_P2.54mm_Vertical, F.Cu at (141.5, 113.5)
- added REF**: PinHeader_1x02_P2.54mm_Vertical, Connector_PinHeader_2.54mm:PinHeader_1x02_P2.54mm_Vertical, F.Cu at (199.5, 113.5)
- added REF**: PinHeader_1x02_P2.54mm_Vertical, Connector_PinHeader_2.54mm:PinHeader_1x02_P2.54mm_Vertical, F.Cu at (264.5, 114.5)
- added SW11: BUTTON_FORCE, Button_Switch_THT:SW_PUSH_6mm_mod, F.Cu at (263.5, 89.5)
- added SW12: SWITCH_MAIN, Button_Switch_THT:SW_DIP_SPSTx01_Slide_9.78x4.72mm_W7.62mm_P2.54mm, F.Cu at (225.9, 80.0)
- added SW13: SWITCH_MAIN, Button_Switch_THT:SW_DIP_SPSTx01_Slide_9.78x4.72mm_W7.62mm_P2.54mm, F.Cu at (105.5, 89.8)
- added SW2: BUTTON_CONFIG, Button_Switch_THT:SW_PUSH_6mm_mod, F.Cu at (189.2, 82.2)
- added SW7: BUTTON_FORCE, Button_Switch_THT:SW_PUSH_6mm_mod, F.Cu at (201.2, 89.2)
- added SW8: SWITCH_MAIN, Button_Switch_THT:SW_DIP_SPSTx01_Slide_9.78x4.72mm_W7.62mm_P2.54mm, F.Cu at (163.1, 78.2)
- added U1: 5V Regulator, Package_TO_SOT_THT:TO-218-3_Vertical, F.Cu at (25.8, 101.3)
- D3: value SOL2_GRN -> SOL1_GRN
- D4: value SOL2_RED -> SOL1_RED
- J2: value SOL2_PORT -> SOL1_PORT
- Q3: value SOL2_NFET -> SOL1_NFET
- R1, R6: value 1kO -> 100O
- R2: value 100 -> 1kO
- R4, R5: value 10kO -> 1kO
- SW10: value SOL2_MASTER -> BUTTON_CONFIG; footprint Button_Switch_THT:SW_DIP_SPSTx01_Slide_6.7x4.1mm_W7.62mm_P2.54mm_LowProfile -> Button_Switch_THT:SW_PUSH_6mm_mod
- SW3: value SOL1_DURA -> DIAL; footprint Rotary_Encoder:RotaryEncoder_Alps_EC11E_Vertical_H20mm -> Button_Switch_THT:RotaryEncoder_Vertical_H20mm
- SW5: value SOL2_DURA -> BUTTON_CONFIG; footprint Rotary_Encoder:RotaryEncoder_Alps_EC11E_Vertical_H20mm -> Button_Switch_THT:SW_PUSH_6mm_mod
- SW6: value SOL2_DELAY -> BUTTON_FORCE; footprint Rotary_Encoder:RotaryEncoder_Alps_EC11E_Vertical_H20mm -> Button_Switch_THT:SW_PUSH_6mm_mod
- moved U1 165.1 mm to (248.8, -40.5)
- moved Q3 130.0 mm to (276.8, 60.3)
- moved D3 112.9 mm to (265.0, 52.0), turned to 0 degrees
- moved SW3 111.9 mm to (45.8, 110.8), turned to -90 degrees
- moved D4 105.2 mm to (251.5, 57.0), turned to 0 degrees
- moved SW10 89.2 mm to (252.5, 82.5), turned to -90 degrees
- moved Q1 88.4 mm to (153.2, 61.8)
- moved SW5 84.4 mm to (129.8, 88.2), turned to -90 degrees
- moved R5 65.8 mm to (118.1, 104.8), turned to 0 degrees
- moved SW6 64.0 mm to (139.2, 94.8)
- moved J2 61.7 mm to (215.5, 104.0), turned to 90 degrees
- moved R2 58.8 mm to (123.8, 83.0), turned to 90 degrees
- moved R6 58.2 mm to (176.9, 69.8), turned to 180 degrees
- moved D5 55.5 mm to (140.5, 62.8), turned to 0 degrees
- moved J3 55.1 mm to (152.2, 104.0), turned to 90 degrees
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Connections:
- net /Microcontroller/5V_OUT renamed Net-(U4-OUT)
- net /Microcontroller/SOL1_RED renamed /Microcontroller/SOL1_WAIT
- D3 pad 1: Net-(D3-K) -> GND
- D5 pad 1: Net-(D5-K) -> GND
- J2 pad 1: Net-(J2-Pin_1) -> /Input Display/12V_R
- J2 pad 2: GND -> Net-(J2-Pin_2)
- J3 pad 1: Net-(J3-Pin_1) -> /Input Display/12V_R
- J3 pad 2: GND -> Net-(J3-Pin_2)
- Q1 pad 1: Net-(J3-Pin_1) -> GND
- Q1 pad 2: VCC -> Net-(J3-Pin_2)
- Q1 pad 3: Net-(Q1-G) -> GND
- Q3 pad 1: Net-(J2-Pin_1) -> GND
- Q3 pad 2: VCC -> Net-(J4-Pin_2)
- Q3 pad 3: Net-(Q3-G) -> GND
- R1 pad 1: Net-(D5-K) -> Net-(R1-Pad1)
- R1 pad 2: Net-(Q1-G) -> /Microcontroller/SOL1_OUT
- R1LED_G1 pad 1: /Solenoid 1 Inputs/OUTPUT -> Net-(R1-Pad1)
- R2 pad 1: /Solenoid 2 Inputs/OUTPUT -> Net-(R1-Pad1)
- R2 pad 2: Net-(D3-K) -> GND
- R3 pad 1: /Solenoid 1 Inputs/OUTPUT -> Net-(R1-Pad1)
- R3 pad 2: Net-(D5-K) -> GND
- R4 pad 1: Net-(D5-K) -> GND
- R4 pad 2: GND -> /Microcontroller/SOL2_SEL
- R5 pad 1: Net-(D3-K) -> GND
- R5 pad 2: GND -> /Microcontroller/SOL1_SEL
- R6 pad 1: Net-(D3-K) -> Net-(R1LED_G2-Pad1)
- R6 pad 2: Net-(Q3-G) -> /Microcontroller/SOL2_OUT
- SW10 pad 1: /Microcontroller/SOL2_GREEN -> unconnected-(SW10-Pad1)
- SW10 pad 2: /Solenoid 2 Inputs/OUTPUT -> unconnected-(SW10-Pad2)
- SW3 pad A: /Microcontroller/SOL1_DURA -> /Input Display/DT
- SW3 pad C: /Microcontroller/SOL1_CLOCK -> /Input Display/CLOCK
- U4 pad 1: VCC -> /Input Display/12V_R
- U4 pad 3: Net-(U4-FB) -> GND
- U4 pad 5: Net-(U4-FB) -> GND
- U4 pad 6: Net-(U4-FB) -> GND
- U4 pad 7: Net-(U4-FB) -> GND
- U4 pad 8: Net-(U4-FB) -> GND
- UC1 pad 11: /Microcontroller/SOL2_RED -> /Microcontroller/SOL1_MAIN
- UC1 pad 12: /Microcontroller/SOL1_GREEN -> /Microcontroller/SOL1_OUT
- UC1 pad 13: /Microcontroller/SOL2_GREEN -> /Microcontroller/SOL1_SEL
- UC1 pad 14: /Microcontroller/SOL1_CONF -> /Microcontroller/SOL2_MAIN
- UC1 pad 15: unconnected-(UC1-PB1-Pad15) -> /Microcontroller/SOL2_OUT
- UC1 pad 16: /Microcontroller/SOL1_CLOCK -> /Microcontroller/SOL2_WAIT
- UC1 pad 17: /Microcontroller/SOL1_DURA -> /Microcontroller/SOL2_SEL
- UC1 pad 18: /Microcontroller/SOL1_DELAY -> /Input Display/SWITCH
- UC1 pad 20: unconnected-(UC1-AVCC-Pad20) -> /Input Display/VCC_E
- UC1 pad 22: Net-(U4-FB) -> GND
- UC1 pad 23: /Microcontroller/SOL2_CONF -> /Microcontroller/SOL3_MAIN
- UC1 pad 24: /Microcontroller/SOL2_DELAY -> /Microcontroller/SOL3_OUT
- UC1 pad 25: /Microcontroller/SOL2_CLOCK -> /Microcontroller/SOL3_WAIT
- UC1 pad 26: /Microcontroller/SOL2_DURA -> /Microcontroller/SOL3_SEL
- UC1 pad 27: /Microcontroller/SDA -> /Input Display/SDA
- UC1 pad 28: /Microcontroller/SCL -> /Input Display/SCL
- UC1 pad 4: /Microcontroller/SOL1_CHECK -> /Input Display/CLOCK
- UC1 pad 5: /Microcontroller/SOL2_CHECK -> /Input Display/DT
- UC1 pad 8: Net-(U4-FB) -> GND
Routing:
- net /Input Display/12V_R: track 0.00 -> 316.4 mm, vias 0 -> 3
- net /Input Display/VCC_E: track 0.00 -> 153.2 mm
- net /Microcontroller/SOL2_DURA: track 126.4 -> 0.00 mm
- net /Microcontroller/SOL2_RED: track 114.6 -> 0.00 mm, vias 1 -> 0
- net /Microcontroller/SOL2_DELAY: track 107.2 -> 0.00 mm, vias 2 -> 0
- net GND: track 78.0 -> 184.5 mm, vias 4 -> 2
- net /Input Display/SWITCH: track 0.00 -> 97.6 mm
- net /Solenoid 2 Inputs/OUTPUT: track 92.5 -> 0.00 mm, vias 1 -> 0
- net /Solenoid 1 Inputs/OUTPUT: track 87.4 -> 0.00 mm, vias 1 -> 0
- net Net-(J2-Pin_2): track 0.00 -> 43.5 mm
- net Net-(J4-Pin_2): track 0.00 -> 42.9 mm
- net VCC: track 42.3 -> 0.00 mm, vias 4 -> 0
- net Net-(J3-Pin_2): track 0.00 -> 41.3 mm
- net /Microcontroller/SOL1_MAIN: track 0.00 -> 37.1 mm
- net /Microcontroller/SOL1_OUT: track 0.00 -> 34.9 mm
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- added copper zone on B.Cu, net GND
