File: hardware/kicad/flowcontrol/flowcontrol.kicad_sch (KiCad schematic)
At the start: 0 parts

Commit message: semi-final updates for the report
Changed lines of the file:
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@@
-	)
-	(junction
-		(at 114.3 68.58)
-		(diameter 0)
-		(color 0 0 0 0)
 	)
 	(junction
@@
 	)
 	(junction
-		(at 100.33 68.58)
-		(diameter 0)
-		(color 0 0 0 0)
-	)
-	(junction
 		(at 34.29 83.82)
 		(diameter 0)
@@
 	)
 	(junction
+		(at 21.59 83.82)
+		(diameter 0)
+		(color 0 0 0 0)
+	)
+	(junction
 		(at 76.2 39.37)
 		(diameter 0)
@@
 	(wire
 		(pts
+			(xy 100.33 67.31) (xy 100.33 62.23)
+		)
+		(stroke
+			(width 0)
+			(type default)
+		)
+	)
+	(wire
+		(pts
 			(xy 26.67 137.16) (xy 26.67 86.36)
 		)
@@
 	(wire
 		(pts
-			(xy 111.76 67.31) (xy 111.76 29.21)
+			(xy 111.76 66.04) (xy 111.76 29.21)
 		)
 		(stroke
@@
 	(wire
 		(pts
-			(xy 24.13 86.36) (xy 26.67 86.36)
+			(xy 21.59 86.36) (xy 26.67 86.36)
 		)
 		(stroke
@@
 	(wire
 		(pts
-			(xy 102.87 62.23) (xy 102.87 67.31)
+			(xy 102.87 62.23) (xy 102.87 66.04)
 		)
 		(stroke
@@
 	(wire
 		(pts
-			(xy 100.33 68.58) (xy 114.3 68.58)
-		)
-		(stroke
-			(width 0)
-			(type default)
-		)
-	)
-	(wire
-		(pts
 			(xy 130.81 71.12) (xy 130.81 120.65)
 		)
@@
 	(wire
 		(pts
-			(xy 58.42 68.58) (xy 100.33 68.58)
+			(xy 58.42 68.58) (xy 132.08 68.58)
 		)
 		(stroke
@@
 	(wire
 		(pts
-			(xy 102.87 67.31) (xy 111.76 67.31)
+			(xy 102.87 66.04) (xy 111.76 66.04)
 		)
 		(stroke
@@
 	(wire
 		(pts
+			(xy 114.3 26.67) (xy 114.3 67.31)
+		)
+		(stroke
+			(width 0)
+			(type default)
+		)
+	)
+	(wire
+		(pts
 			(xy 167.64 83.82) (xy 167.64 120.65)
 		)
@@
 	(wire
 		(pts
+			(xy 114.3 67.31) (xy 100.33 67.31)
+		)
+		(stroke
+			(width 0)
+			(type default)
+		)
+	)
+	(wire
+		(pts
 			(xy 165.1 123.19) (xy 170.18 123.19)
 		)
@@
 	(wire
 		(pts
-			(xy 105.41 66.04) (xy 109.22 66.04)
+			(xy 105.41 64.77) (xy 109.22 64.77)
 		)
 		(stroke
@@
 	(wire
 		(pts
-			(xy 105.41 62.23) (xy 105.41 66.04)
+			(xy 105.41 62.23) (xy 105.41 64.77)
 		)
 		(stroke
@@
 	(wire
 		(pts
-			(xy 114.3 68.58) (xy 132.08 68.58)
-		)
-		(stroke
-			(width 0)
-			(type default)
-		)
-	)
-	(wire
-		(pts
 			(xy 110.49 137.16) (xy 26.67 137.16)
 		)
@@
 	(wire
 		(pts
-			(xy 100.33 62.23) (xy 100.33 68.58)
-		)
-		(stroke
-			(width 0)
-			(type default)
-		)
-	)
-	(wire
-		(pts
-			(xy 24.13 83.82) (xy 34.29 83.82)
+			(xy 21.59 83.82) (xy 34.29 83.82)
 		)
 		(stroke
@@
 	(wire
 		(pts
-			(xy 114.3 68.58) (xy 114.3 26.67)
-		)
-		(stroke
-			(width 0)
-			(type default)
-		)
-	)
-	(wire
-		(pts
 			(xy 76.2 58.42) (xy 76.2 120.65)
 		)
@@
 	(wire
 		(pts
-			(xy 109.22 66.04) (xy 109.22 31.75)
+			(xy 109.22 64.77) (xy 109.22 31.75)
 		)
 		(stroke
@@
 	)
 	(symbol
-		(lib_id "power:GND")
-		(at 24.13 83.82 270)
+		(lib_id "power:PWR_FLAG")
+		(at 21.59 83.82 0)
 		(unit 1)
 		(exclude_from_sim no)
@@
 		(dnp no)
 		(fields_autoplaced yes)
-		(property "Reference" "#PWR06"
-			(at 17.78 83.82 0)
+		(property "Reference" "#FLG02"
+			(at 21.59 81.915 0)
 			(effects
 				(font
@@
 			)
 		)
-		(property "Value" "GND"
-			(at 20.32 83.8199 90)
-			(effects
-				(font
-					(size 1.27 1.27)
-				)
-				(justify right)
+		(property "Value" "PWR_FLAG"
+			(at 21.59 78.74 0)
+			(effects
+				(font
+					(size 1.27 1.27)
+				)
 			)
 		)
 		(property "Footprint" ""
-			(at 24.13 83.82 0)
+			(at 21.59 83.82 0)
 			(effects
 				(font
@@
 			)
 		)
-		(property "Datasheet" ""
-			(at 24.13 83.82 0)
+		(property "Datasheet" "~"
+			(at 21.59 83.82 0)
 			(effects
 				(font
@@
 			)
 		)
-		(property "Description" "Power symbol creates a global label with name \"GND\" , ground"
-			(at 24.13 83.82 0)
+		(property "Description" "Special symbol for telling ERC where power comes from"
+			(at 21.59 83.82 0)
 			(effects
 				(font
@@
 		)
 		(instances
-			(project "flowcontrol"
+			(project ""
 				(path "/c8fb4b8d-0361-4798-b029-ef8709a5481b"
-					(reference "#PWR06")
+					(reference "#FLG02")
 					(unit 1)
 				)
@@
 	)
 	(symbol
-		(lib_id "power:VCC")
-		(at 24.13 86.36 90)
+		(lib_id "power:GND")
+		(at 21.59 83.82 270)
 		(unit 1)
 		(exclude_from_sim no)
@@
 		(dnp no)
 		(fields_autoplaced yes)
-		(property "Reference" "#PWR05"
-			(at 27.94 86.36 0)
+		(property "Reference" "#PWR01"
+			(at 15.24 83.82 0)
 			(effects
 				(font
@@
 			)
 		)
-		(property "Value" "VCC"
-			(at 20.32 86.3599 90)
-			(effects
-				(font
-					(size 1.27 1.27)
-				)
-				(justify left)
+		(property "Value" "GND"
+			(at 17.78 83.8199 90)
+			(effects
+				(font
+					(size 1.27 1.27)
+				)
+				(justify right)
 			)
 		)
 		(property "Footprint" ""
-			(at 24.13 86.36 0)
+			(at 21.59 83.82 0)
 			(effects
 				(font
@@
 		)
 		(property "Datasheet" ""
-			(at 24.13 86.36 0)
+			(at 21.59 83.82 0)
 			(effects
 				(font
@@
 			)
 		)
-		(property "Description" "Power symbol creates a global label with name \"VCC\""
-			(at 24.13 86.36 0)
+		(property "Description" "Power symbol creates a global label with name \"GND\" , ground"
+			(at 21.59 83.82 0)
 			(effects
 				(font
@@
 			(project ""
 				(path "/c8fb4b8d-0361-4798-b029-ef8709a5481b"
-					(reference "#PWR05")
+					(reference "#PWR01")
 					(unit 1)
 				)
+			)
+		)
+	)
+	(symbol
+		(lib_id "power:PWR_FLAG")
+		(at 21.59 86.36 90)
+		(unit 1)
+		(exclude_from_sim no)
+		(in_bom yes)
+		(on_board yes)
+		(dnp no)
+		(fields_autoplaced yes)
+		(property "Reference" "#FLG01"
+			(at 19.685 86.36 0)
+			(effects
+				(font
+					(size 1.27 1.27)
+				)
+				(hide yes)
+			)
+		)
+		(property "Value" "12V"
+			(at 17.78 86.3599 90)
+			(effects
+				(font
+					(size 1.27 1.27)
+				)
+				(justify left)
+			)
+		)
+		(property "Footprint" ""
+			(at 21.59 86.36 0)
+			(effects
+				(font
+					(size 1.27 1.27)
+				)
+				(hide yes)
+			)
+		)
+		(property "Datasheet" "~"
+			(at 21.59 86.36 0)
+			(effects
+				(font
+					(size 1.27 1.27)
+				)
+				(hide yes)
+			)
+		)
+		(property "Description" "Special symbol for telling ERC where power comes from"
+			(at 21.59 86.36 0)
+			(effects
+				(font
+					(size 1.27 1.27)
+				)
+				(hide yes)
+			)
+		)
+		(pin "1"
+		)
+		(instances
+			(project ""
+				(path "/c8fb4b8d-0361-4798-b029-ef8709a5481b"
+					(reference "#FLG01")
+					(unit 1)
+				)
