File: hardware/kicad/flowcontrol/sol1_output.kicad_sch (KiCad schematic)
At the start: 7 parts, among them J3 SOL1_PORT, Q3 SOL1_NPN

Commit message: Schemiatic update
Parts:
- removed Q3: SOL1_NPN, symbol Simulation_SPICE:NPN
- added Q1: SOL1_NFET, Package_TO_SOT_SMD:SOT-23, symbol Transistor_FET:MMBFJ113
- added R1: 1kO, Resistor_THT:R_Axial_DIN0309_L9.0mm_D3.2mm_P15.24mm_Horizontal, symbol Device:R
- added R4: 10kO, Resistor_THT:R_Axial_DIN0309_L9.0mm_D3.2mm_P15.24mm_Horizontal, symbol Device:R
- D5, D6: footprint (none) -> LED_THT:LED_Oval_W5.2mm_H3.8mm
- J3: footprint (none) -> Connector_PinSocket_2.00mm:PinSocket_1x02_P2.00mm_Vertical
- R1LED_G1, R1LED_R1, R3: footprint (none) -> Resistor_THT:R_Axial_DIN0309_L9.0mm_D3.2mm_P15.24mm_Horizontal
Connections:
- net 12V_IN: now also Q1.2 (S)
- net GND: now also R4.2
- net at J3.1 (Pin_1): now also Q1.1 (D)
- net at D5.1 (K), R3.2: now also R1.1, R4.1
- new net: Q1.3 (G), R1.2
Other:
- moved on the sheet: D5, D6, R1LED_G1, R1LED_R1, R3

Commit message: Updated KiCad schematic to final rendition
Parts:
- removed R4: 10kO, Resistor_THT:R_Axial_DIN0309_L9.0mm_D3.2mm_P15.24mm_Horizontal, symbol Device:R
- added R2, R5: 1kO, Resistor_THT:R_Axial_DIN0309_L9.0mm_D3.2mm_P15.24mm_Horizontal, symbol Device:R
- added SW2: BUTTON_CONFIG, symbol Switch:SW_Push_Dual
- added SW6: BUTTON_FORCE, symbol Switch:SW_Push_Dual
- added SW8: SWITCH_MAIN, symbol Switch:SW_SPST
- R1: value 1kO -> 100O
- renumbered Q1 to Q2
Connections:
- net GND: now also D5.1 (K), Q2.1 (D), Q2.3 (G), R3.2, R2.2, R5.1; no longer J3.2 (Pin_2)
- net TRIGGER: now also R1.2; no longer R1LED_G1.1, R3.1
- net 12V_SUPPLY: now reaches J3.1 (Pin_1)
- net 12V_SUPPLY: no longer Q2.1 (D)
- net 12V_IN: no longer names the net of Q2.2 (S)
- net 12V_IN: now also J3.2 (Pin_2)
- new net: R1.1, R1LED_G1.1, R2.1, R3.1, SW6.2
- new net 5V: SW2.4, SW6.1, SW8.2 (B)
- new net MAIN: SW8.1 (A)
- new net SETTING: R5.2, SW2.3
- no-connect marks 0 -> 2
Other:
- moved on the sheet: D5, D6, J3, Q2, R1, R1LED_G1, R1LED_R1, R3

Commit message: labeled the old pcb old
Parts:
- renumbered D5 to D1, D6 to D2, J3 to J2, R1LED_G1 to R1LED_G2, R1LED_R1 to R1LED_R2, R5 to R4, R1 to R6, R2 to R7, R3 to R8, SW6 to SW7
Connections:
- no-connect marks 2 -> 4
Changed lines of the file:
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@@
+	)
+	(no_connect
+		(at 46.99 25.4)
 	)
 	(no_connect
 		(at 36.83 58.42)
+	)
+	(no_connect
+		(at 36.83 25.4)
 	)
 	(no_connect
@@
 		(on_board yes)
 		(dnp no)
-		(property "Reference" "R1LED_G1"
+		(property "Reference" "R1LED_G2"
 			(at 51.054 49.784 0)
 			(effects
@@
 					(unit 1)
 				)
+				(path "/c8fb4b8d-0361-4798-b029-ef8709a5481b/e7501852-2e13-483b-b108-2a6b83c28583"
+					(reference "SW13")
+					(unit 1)
+				)
 			)
 		)
@@
 		(on_board yes)
 		(dnp no)
-		(property "Reference" "J3"
+		(property "Reference" "J2"
 			(at 80.01 93.3449 90)
 			(effects
@@
 					(unit 1)
 				)
+				(path "/c8fb4b8d-0361-4798-b029-ef8709a5481b/e7501852-2e13-483b-b108-2a6b83c28583"
+					(reference "Q1")
+					(unit 1)
+				)
 			)
 		)
@@
 		(on_board yes)
 		(dnp no)
-		(property "Reference" "D6"
+		(property "Reference" "D2"
 			(at 85.09 58.42 90)
 			(effects
@@
 		(dnp no)
 		(fields_autoplaced yes)
-		(property "Reference" "R1LED_R1"
+		(property "Reference" "R1LED_R2"
 			(at 81.28 49.5299 0)
 			(effects
@@
 		(on_board yes)
 		(dnp no)
-		(property "Reference" "R3"
+		(property "Reference" "R8"
 			(at 64.262 49.784 0)
 			(effects
@@
 		(on_board yes)
 		(dnp no)
-		(property "Reference" "R1"
+		(property "Reference" "R6"
 			(at 38.862 33.782 90)
 			(effects
@@
 					(unit 1)
 				)
+				(path "/c8fb4b8d-0361-4798-b029-ef8709a5481b/e7501852-2e13-483b-b108-2a6b83c28583"
+					(reference "SW5")
+					(unit 1)
+				)
 			)
 		)
@@
 		(on_board yes)
 		(dnp no)
-		(property "Reference" "R5"
+		(property "Reference" "R4"
 			(at 26.162 30.734 0)
 			(effects
@@
 		(on_board yes)
 		(dnp no)
-		(property "Reference" "R2"
+		(property "Reference" "R7"
 			(at 43.942 62.484 0)
 			(effects
@@
 		(on_board yes)
 		(dnp no)
-		(property "Reference" "D5"
+		(property "Reference" "D1"
 			(at 57.15 58.42 90)
 			(effects
@@
 		(on_board yes)
 		(dnp no)
-		(property "Reference" "SW6"
+		(property "Reference" "SW7"
 			(at 30.226 52.832 0)
 			(effects

Commit message: semi-final updates for the report
Parts:
- SW2, SW7: footprint (none) -> Button_Switch_THT:SW_PUSH_6mm_mod
- SW8: footprint (none) -> Button_Switch_THT:SW_DIP_SPSTx01_Slide_9.78x4.72mm_W7.62mm_P2.54mm
Changed lines of the file:
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@@
 			)
 		)
-		(property "Footprint" ""
+		(property "Footprint" "Button_Switch_THT:SW_DIP_SPSTx01_Slide_9.78x4.72mm_W7.62mm_P2.54mm"
 			(at 59.69 40.64 0)
 			(effects
@@
 			)
 		)
-		(property "Footprint" ""
+		(property "Footprint" "Button_Switch_THT:SW_PUSH_6mm_mod"
 			(at 41.91 20.32 0)
 			(effects
@@
 			)
 		)
-		(property "Footprint" ""
+		(property "Footprint" "Button_Switch_THT:SW_PUSH_6mm_mod"
 			(at 41.91 48.26 0)
 			(effects
